Commit message: Imported upstream version '1.0.6' of 'upstream'

File: rb1_base_description/robots/rb1_base_platform_standalone.urdf.xacro (robot description, xacro)
@@ -6,10 +6,18 @@
 	<!-- First we import all posible elements defined in the urdf.xacro files. All these elements are defined as macro:xacros -->
 	<!-- Import RB1 base elements -->
-    	<xacro:include filename="$(find rb1_base_description)/urdf/bases/rb1_base.urdf.xacro" />
+    <xacro:include filename="$(find rb1_base_description)/urdf/bases/rb1_base.urdf.xacro" />
+    <gazebo>
+      <plugin name="ros_control" filename="libgazebo_ros_control.so">
+        <robotNamespace>/rb1</robotNamespace>
+        <robotParam>robot_description</robotParam>
+        <controlPeriod>0.001</controlPeriod>
+	    <robotSimType>gazebo_ros_control/DefaultRobotHWSim</robotSimType>
+      </plugin>
+    </gazebo>
 	<!-- Import RB1 wheels -->
 	<xacro:include filename="$(find rb1_base_description)/urdf/wheels/rubber_wheel.urdf.xacro" />
 	<xacro:include filename="$(find rb1_base_description)/urdf/wheels/omni_wheel.urdf.xacro" />
 	<!-- Import all available sensors -->
-    	<xacro:include filename="$(find robotnik_sensors)/urdf/all_sensors.urdf.xacro"/>
+    <xacro:include filename="$(find robotnik_sensors)/urdf/all_sensors.urdf.xacro"/>
 	<!-- ***************** -->
 	<!-- Global parameters -->
@@ -60,7 +68,7 @@
 		<origin xyz="0.210 0.0 0.305" rpy="0 0 0"/>
 	</xacro:sensor_hokuyo_utm30lx -->
-	<!-- xacro:sensor_hokuyo_urg04lx name="hokuyo1" parent="base_link">
-		<origin xyz="0.220 0.0 0.170" rpy="0 3.1416 3.1416"/>
-	</xacro:sensor_hokuyo_urg04lx -->
+    <!-- xacro:sensor_hokuyo_urg04lx name="hokuyo1" parent="base_link">
+        <origin xyz="0.220 0.0 0.170" rpy="0 3.1416 3.1416"/>
+    </xacro:sensor_hokuyo_urg04lx -->
 	<!-- xacro:sensor_hokuyo_ust10lx name="hokuyo" parent="base_link">
 		<origin xyz="0.223 0.0 0.159" rpy="0 0 0"/>
@@ -72,6 +80,12 @@
 		<origin xyz="-0.18 0.0 0.170" rpy="0 0 0"/>
 	</xacro:sensor_imu>
-	<xacro:sensor_orbbec_astra name="orbbec_astra" parent="base_link">
-		<origin xyz="0.234 0.0125 0.107" rpy="0 0 0"/>
-	</xacro:sensor_orbbec_astra>
+    <!-- xacro:sensor_orbbec_astra name="orbbec_astra" parent="base_link">
+        <origin xyz="0.234 0.0125 0.107" rpy="0 0 0"/>
+    </xacro:sensor_orbbec_astra -->
+    <xacro:sensor_orbbec_astra name="orbbec_astra" parent="base_link">
+        <origin xyz="0.234 0.0125 0.107" rpy="0 0 0"/>
+    </xacro:sensor_orbbec_astra>
+    <!-- xacro:sensor_kinect name="kinect" parent="base_link">
+        <origin xyz="0.6 0.0 0.102" rpy="0 0 0"/>
+    </xacro:sensor_kinect -->
 </robot>

File: rb1_base_description/urdf/bases/rb1_base.gazebo.xacro (robot description, xacro)
@@ -2,5 +2,5 @@
 <robot xmlns:xacro="http://ros.org/wiki/xacro">
   <!-- ros control plugin -->
-  <xacro:macro name="ros_control">
+  <!-- xacro:macro name="ros_control">
     <gazebo>
       <plugin name="ros_control" filename="libgazebo_ros_control.so">
@@ -11,5 +11,5 @@
       </plugin>
     </gazebo>
-  </xacro:macro>
+	</xacro:macro -->
 	<!-- differential drive plugin -->
 	<xacro:macro name="diff_drive">
@@ -18,6 +18,6 @@
 	    <alwaysOn>true</alwaysOn>
         <updateRate>50.0</updateRate>
-        <!--leftJoint>joint_left_wheel</leftJoint>
-        <rightJoint>joint_right_wheel</rightJoint-->
+        <!-- leftJoint>joint_left_wheel</leftJoint>
+        <rightJoint>joint_right_wheel</rightJoint -->
         <leftJoint>joint_right_wheel</leftJoint>
         <rightJoint>joint_left_wheel</rightJoint>
@@ -32,5 +32,5 @@
         <!-- robotNamespace></robotNamespace -->
         <rosDebugLevel>na</rosDebugLevel>
-        <publishWheelTF>true</publishWheelTF>
+        <publishWheelTF>false</publishWheelTF>
         <publishWheelJointState>false</publishWheelJointState>
         <wheelAcceleration>0</wheelAcceleration>
@@ -39,5 +39,4 @@
         <odometrySource>world</odometrySource>
         <publishTf>1</publishTf>
-	<legacyMode>false</legacyMode>
 	</plugin>
 	</gazebo>

File: rb1_base_description/urdf/bases/rb1_base.urdf.xacro (robot description, xacro)
@@ -1,5 +1,5 @@
 <?xml version="1.0"?>
 <robot name="rb1_base" xmlns:xacro="http://www.ros.org/wiki/xacro">
-  <xacro:include filename="$(find rb1_base_description)/urdf/bases/rb1_base.gazebo.xacro" />
+  <!-- xacro:include filename="$(find rb1_base_description)/urdf/bases/rb1_base.gazebo.xacro" / -->
   <xacro:macro name="rb1_base" params="name publish_bf hq">
   <!-- Robot mechanical and motor parameters -->

File: rb1_base_description/urdf/wheels/omni_wheel.urdf.xacro (robot description, xacro)
@@ -3,7 +3,7 @@
   <xacro:property name="M_PI" value="3.1415926535897931" />
   <!-- Wheels -->
-  <xacro:property name="omni_wheel_radius" value="0.051" />
-  <xacro:property name="omni_wheel_height" value="0.040" />
-  <xacro:property name="omni_wheel_mass" value="0.3" /> <!-- in kg-->
+  <property name="omni_wheel_radius" value="0.051" />
+  <property name="omni_wheel_height" value="0.040" />
+  <property name="omni_wheel_mass" value="0.3" /> <!-- in kg-->
   <xacro:macro name="cylinder_inertia" params="m r h">
     <inertia  ixx="${m*(3*r*r+h*h)/12}" ixy = "0" ixz = "0"
@@ -17,5 +17,5 @@
       <parent link="${parent}"/>
       <child link="${name}_wheel"/>
-      <xacro:insert_block name="origin" />
+      <insert_block name="origin" />
       <axis xyz="0 1 0" rpy="0 0 0" />
       <limit effort="100" velocity="100"/>

File: rb1_base_description/urdf/wheels/omni_wheel_v1.urdf.xacro (robot description, xacro)
@@ -3,7 +3,7 @@
   <xacro:property name="M_PI" value="3.1415926535897931" />
   <!-- Wheels -->
-  <xacro:property name="omni_wheel_radius" value="0.051" />
-  <xacro:property name="omni_wheel_height" value="0.040" />
-  <xacro:property name="omni_wheel_mass" value="0.3" /> <!-- in kg-->
+  <property name="omni_wheel_radius" value="0.051" />
+  <property name="omni_wheel_height" value="0.040" />
+  <property name="omni_wheel_mass" value="0.3" /> <!-- in kg-->
   <xacro:macro name="cylinder_inertia" params="m r h">
     <inertia  ixx="${m*(3*r*r+h*h)/12}" ixy = "0" ixz = "0"
@@ -17,5 +17,5 @@
       <parent link="${parent}"/>
       <child link="${name}_wheel"/>
-      <xacro:insert_block name="origin" />
+      <insert_block name="origin" />
       <axis xyz="0 1 0" rpy="0 0 0" />
       <limit effort="100" velocity="100"/>

File: rb1_base_description/urdf/wheels/rubber_wheel.urdf.xacro (robot description, xacro)
@@ -3,7 +3,7 @@
   <xacro:property name="M_PI" value="3.1415926535897931" />
   <!-- Wheels -->
-  <xacro:property name="wheel_radius" value="0.076" />
-  <xacro:property name="wheel_height" value="0.025" />
-  <xacro:property name="wheel_mass" value="1.0" /> <!-- in kg-->
+  <property name="wheel_radius" value="0.076" />
+  <property name="wheel_height" value="0.025" />
+  <property name="wheel_mass" value="1.0" /> <!-- in kg-->
   <xacro:macro name="cylinder_inertia" params="m r h">
     <inertia  ixx="${m*(3*r*r+h*h)/12}" ixy = "0" ixz = "0"
@@ -16,5 +16,5 @@
       <parent link="${parent}"/>
       <child link="${name}_wheel"/>
-      <xacro:insert_block name="origin" />
+      <insert_block name="origin" />
       <axis xyz="0 1 0" rpy="0 0 0" />
       <limit effort="100" velocity="100"/>
