Commit message: Imported upstream version '1.1.0' of 'upstream'

File: rb1_base_description/urdf/bases/rb1_base.gazebo.xacro (robot description, xacro)
@@ -2,5 +2,5 @@
 <robot xmlns:xacro="http://ros.org/wiki/xacro">
   <!-- ros control plugin -->
-  <!-- xacro:macro name="ros_control">
+  <xacro:macro name="ros_control">
     <gazebo>
       <plugin name="ros_control" filename="libgazebo_ros_control.so">
@@ -11,5 +11,5 @@
       </plugin>
     </gazebo>
-	</xacro:macro -->
+  </xacro:macro>
 	<!-- differential drive plugin -->
 	<xacro:macro name="diff_drive">
@@ -18,6 +18,6 @@
 	    <alwaysOn>true</alwaysOn>
         <updateRate>50.0</updateRate>
-        <!-- leftJoint>joint_left_wheel</leftJoint>
-        <rightJoint>joint_right_wheel</rightJoint -->
+        <!--leftJoint>joint_left_wheel</leftJoint>
+        <rightJoint>joint_right_wheel</rightJoint-->
         <leftJoint>joint_right_wheel</leftJoint>
         <rightJoint>joint_left_wheel</rightJoint>
@@ -32,5 +32,5 @@
         <!-- robotNamespace></robotNamespace -->
         <rosDebugLevel>na</rosDebugLevel>
-        <publishWheelTF>false</publishWheelTF>
+        <publishWheelTF>true</publishWheelTF>
         <publishWheelJointState>false</publishWheelJointState>
         <wheelAcceleration>0</wheelAcceleration>
@@ -39,4 +39,5 @@
         <odometrySource>world</odometrySource>
         <publishTf>1</publishTf>
+	<legacyMode>false</legacyMode>
 	</plugin>
 	</gazebo>

File: rb1_base_description/urdf/bases/rb1_base.urdf.xacro (robot description, xacro)
@@ -1,5 +1,5 @@
 <?xml version="1.0"?>
 <robot name="rb1_base" xmlns:xacro="http://www.ros.org/wiki/xacro">
-  <!-- xacro:include filename="$(find rb1_base_description)/urdf/bases/rb1_base.gazebo.xacro" / -->
+  <xacro:include filename="$(find rb1_base_description)/urdf/bases/rb1_base.gazebo.xacro" />
   <xacro:macro name="rb1_base" params="name publish_bf hq">
   <!-- Robot mechanical and motor parameters -->
